Commit message: Two-dimensional pendulum implemented

File: robots/franka_pole_2D.xacro (robot description, xacro)
@@ -51,5 +51,5 @@
       <origin xyz="0 0 0" rpy="0 0 0"/>
       <geometry>
-        <mesh filename="package://franka_pole/meshes/visual/1D_lower.dae"/>
+        <mesh filename="package://franka_pole/meshes/visual/2D_lower.dae"/>
       </geometry>
     </visual>
@@ -63,6 +63,31 @@
     </inertial>
   </link>
+  <joint name="$(arg arm_id)_pole_joint_y" type="revolute">
+    <parent link="$(arg arm_id)_pole_link_lower"/>
+    <child link="$(arg arm_id)_pole_link_middle"/>
+    <origin xyz="0 0 0" rpy="0 0 0"/>
+    <axis xyz="0 1 0"/>
+    <limit velocity="1000000" lower="${-20*pi/180}" effort="0" upper="${20*pi/180}" />
+    <dynamics damping="0.0"/>
+  </joint>
+  <!-- Middle bearing -->
+  <link name="$(arg arm_id)_pole_link_middle">
+    <visual>
+      <origin xyz="0 0 0" rpy="0 0 0"/>
+      <geometry>
+        <mesh filename="package://franka_pole/meshes/visual/2D_middle.dae"/>
+      </geometry>
+    </visual>
+    <inertial>
+      <origin xyz="0 0 0" rpy="0 0 0"/>
+      <mass value="0.1"/>
+      <inertia
+      ixx="0.0" ixy="0.0" ixz="0.0"
+      iyy="0.0" iyz="0.0"
+      izz="0.0"/>
+    </inertial>
+  </link>
   <joint name="$(arg arm_id)_pole_joint_x" type="revolute">
-    <parent link="$(arg arm_id)_pole_link_lower"/>
+    <parent link="$(arg arm_id)_pole_link_middle"/>
     <child link="$(arg arm_id)_pole_link_upper"/>
     <origin xyz="0 0 0" rpy="0 0 0"/>
@@ -81,5 +106,5 @@
     <visual>
       <geometry>
-        <mesh filename="package://franka_pole/meshes/visual/1D_upper.dae"/>
+        <mesh filename="package://franka_pole/meshes/visual/2D_upper.dae"/>
       </geometry>
     </visual>
@@ -115,4 +140,13 @@
     </inertial>
   </link>
+  <transmission name="$(arg arm_id)_pole_joint_y_transmission">
+    <type>transmission_interface/SimpleTransmission</type>
+    <joint name="$(arg arm_id)_pole_joint_y">
+      <hardwareInterface>hardware_interface/PositionJointInterface</hardwareInterface>
+    </joint>
+    <actuator name="$(arg arm_id)_pole_joint_y_motor">
+      <hardwareInterface>hardware_interface/PositionJointInterface</hardwareInterface>
+    </actuator>
+  </transmission>
   <transmission name="$(arg arm_id)_pole_joint_x_transmission">
     <type>transmission_interface/SimpleTransmission</type>

Commit message: Acceleration control improved

File: robots/franka_pole_2D.xacro (robot description, xacro)
@@ -42,5 +42,5 @@
   <!-- Connection -->
   <joint name="$(arg arm_id)_pole_joint_connection" type="fixed">
-    <origin xyz="0.071 -0.071 0.03" rpy="${pi} 0 ${-pi/4}" />
+    <origin xyz="0.071 -0.071 0.0" rpy="${pi} 0 ${-pi/4}" />
     <parent link="$(arg arm_id)_link8" />
     <child  link="$(arg arm_id)_pole_link_lower" />

Commit message: Euler angles corrected

File: robots/franka_pole_2D.xacro (robot description, xacro)
@@ -36,4 +36,5 @@
   <!-- Pendulum -->
   <xacro:property name="lower_mass" value="0.5" />
+  <xacro:property name="middle_mass" value="0.05" />
   <xacro:property name="upper_mass" value="0.1" />
   <xacro:property name="ball_mass" value="0.1" />
@@ -83,5 +84,5 @@
     <inertial>
       <origin xyz="0 0 0" rpy="0 0 0"/>
-      <mass value="0.1"/>
+      <mass value="${middle_mass}"/>
       <inertia
       ixx="0.0" ixy="0.0" ixz="0.0"

Commit message: 2D balancing almost working

File: robots/franka_pole_2D.xacro (robot description, xacro)
@@ -71,5 +71,5 @@
     <origin xyz="0 0 0" rpy="0 0 0"/>
     <axis xyz="0 1 0"/>
-    <limit velocity="1000000" lower="${-10*pi/180}" effort="0" upper="${10*pi/180}" />
+    <limit velocity="1000000" lower="${-30*pi/180}" effort="0" upper="${30*pi/180}" />
     <dynamics damping="0.0"/>
   </joint>
@@ -96,5 +96,5 @@
     <origin xyz="0 0 0.012" rpy="0 0 0"/>
     <axis xyz="1 0 0"/>
-    <limit velocity="1000000" lower="${-10*pi/180}" effort="0" upper="${10*pi/180}" />
+    <limit velocity="1000000" lower="${-30*pi/180}" effort="0" upper="${30*pi/180}" />
     <dynamics damping="0.0"/>
   </joint>
