Commit message: New pendulum model added

File: robots/franka_pole_2Db.xacro (robot description, xacro)
@@ -45,14 +45,14 @@
       <origin xyz="0 0 0" rpy="0 0 0"/>
       <geometry>
-        <mesh filename="package://franka_pole/meshes/visual/2D_lower.dae"/>
+        <mesh filename="package://franka_pole/meshes/visual/2Db_lower.dae"/>
       </geometry>
     </visual>
     <inertial>
-      <origin xyz="-0.05109889873590216 2.087955225371467e-05 -0.09641756504956266" rpy="0 0 0"/>
-      <mass value="0.3291666816221097"/>
+      <origin xyz="0.0 -0.03161502390972815 -0.06659192458617054" rpy="0 0 0"/>
+      <mass value="0.27322280135974475"/>
       <inertia
-      ixx="0.0019391504246096141" ixy="-1.2810025473031176e-07" ixz="-0.00018658257593334764"
-      iyy="0.0032282596099721715" iyz="-2.76251743233805e-07"
-      izz="0.002428110536000401"/>
+      ixx="0.0028058366276666187" ixy="0.0" ixz="0.0"
+      iyy="0.0016993982151537815" iyz="-8.877913787029444e-05"
+      izz="0.002116794356382879"/>
     </inertial>
   </link>
@@ -62,22 +62,12 @@
     <origin xyz="0 0 0" rpy="0 0 0"/>
     <axis xyz="0 1 0"/>
-    <limit velocity="1000000" lower="${0*pi/180}" effort="0" upper="${60*pi/180}" />
+    <limit velocity="1000000" lower="${-30*pi/180}" effort="0" upper="${30*pi/180}" />
     <dynamics damping="0.0"/>
   </joint>
   <!-- Middle bearing -->
   <link name="$(arg arm_id)_pole_link_middle">
-    <visual>
-      <origin xyz="0 0 0" rpy="0 0 0"/>
-      <geometry>
-        <mesh filename="package://franka_pole/meshes/visual/2D_middle.dae"/>
-      </geometry>
-    </visual>
     <inertial>
-      <origin xyz="0.0 6.359054534633294e-09 0.006000000469716085" rpy="0 0 0"/>
-      <mass value="0.01583948395827795"/>
-      <inertia
-      ixx="2.2608411674142452e-05" ixy="0.0" ixz="0.0"
-      iyy="2.2608411674142462e-05" iyz="0.0"
-      izz="1.612722485663805e-05"/>
+      <origin xyz="0.0 0.0 0.0" rpy="0 0 0"/>
+      <mass value="0.001"/>
     </inertial>
   </link>
@@ -85,5 +75,5 @@
     <parent link="$(arg arm_id)_pole_link_middle"/>
     <child link="$(arg arm_id)_pole_link_upper"/>
-    <origin xyz="0 0 0.012" rpy="0 0 0"/>
+    <origin xyz="0 0 0" rpy="0 0 0"/>
     <axis xyz="1 0 0"/>
     <limit velocity="1000000" lower="${-30*pi/180}" effort="0" upper="${30*pi/180}" />
@@ -93,28 +83,22 @@
   <link name="$(arg arm_id)_pole_link_upper">
     <visual>
-      <origin xyz="0 0 -0.012" rpy="0 0 0"/>
+      <origin xyz="0 0 0" rpy="0 0 0"/>
       <geometry>
-        <mesh filename="package://franka_pole/meshes/visual/2D_upper.dae"/>
+        <mesh filename="package://franka_pole/meshes/visual/2Db_upper.dae"/>
       </geometry>
     </visual>
     <visual>
-      <origin xyz="0 0 ${0.06 + 0.65/2}" rpy="0 0 0"/>
+      <origin xyz="0 0 ${0.039 + 0.5/2}" rpy="0 0 0"/>
       <geometry>
-        <cylinder length="0.65" radius="0.005"/>
-      </geometry>
-    </visual>
-    <visual>
-      <origin xyz="0 0 0.43" rpy="0 0 0"/>
-      <geometry>
-        <sphere radius="0.0275"/>
+        <cylinder length="0.5" radius="0.005"/>
       </geometry>
     </visual>
     <inertial>
-      <origin xyz="-6.25914508960298e-05 2.6377566995216277e-07 ${0.18536862521254435 - 0.012}" rpy="0 0 0"/>
-      <mass value="0.13492793369531808"/>
+      <origin xyz="0.0 0.0 0.35075520003248506" rpy="0 0 0"/>
+      <mass value="0.03241958003770816"/>
       <inertia
-      ixx="0.005511654978105017" ixy="0.0" ixz="-9.981512278924966e-07"
-      iyy="0.005311406380325907" iyz="6.358922261996068e-09"
-      izz="0.00036275792557540116"/>
+      ixx="0.001036931649741803" ixy="0.0" ixz="0.0"
+      iyy="0.001036931649741803" iyz="0.0"
+      izz="1.109395012820758e-05"/>
     </inertial>
   </link>
