Commit message: Structured

File: robots/franka_pole.xacro (robot description, xacro)
@@ -51,5 +51,5 @@
       <origin xyz="0 0 0" rpy="0 0 0"/>
       <geometry>
-        <mesh filename="package://franka_pole/visual/lower_bearing.dae"/>
+        <mesh filename="package://franka_pole/meshes/visual/lower_bearing.dae"/>
       </geometry>
     </visual>
@@ -81,5 +81,5 @@
     <visual>
       <geometry>
-        <mesh filename="package://franka_pole/visual/upper_bearing.dae"/>
+        <mesh filename="package://franka_pole/meshes/visual/upper_bearing.dae"/>
       </geometry>
     </visual>

Commit message: All controllers working

File: robots/franka_pole.xacro (robot description, xacro)
@@ -36,5 +36,5 @@
   <xacro:property name="upper_mass" value="0.1" />
   <xacro:property name="ball_mass" value="0.1" />
-  <xacro:property name="beam_mass" value="0.5" />
+  <xacro:property name="beam_mass" value="0.05" />
   <xacro:property name="beam_length" value="0.6" />
   <xacro:property name="beam_radius" value="0.01" />

Commit message: Reset implemented

File: robots/franka_pole.xacro (robot description, xacro)
@@ -29,4 +29,6 @@
       <controlPeriod>0.001</controlPeriod>
       <robotSimType>franka_gazebo/FrankaHWSim</robotSimType>
+    </plugin>
+    <plugin name="franka_pole_plugin" filename="libfranka_pole_plugin.so">
     </plugin>
     <self_collide>true</self_collide>

File: robots/franka_pole_2D.xacro (robot description, xacro)
@@ -91,5 +91,5 @@
     <parent link="$(arg arm_id)_pole_link_middle"/>
     <child link="$(arg arm_id)_pole_link_upper"/>
-    <origin xyz="0 0 0" rpy="0 0 0"/>
+    <origin xyz="0 0 0.012" rpy="0 0 0"/>
     <axis xyz="1 0 0"/>
     <limit velocity="1000000" lower="${-20*pi/180}" effort="0" upper="${20*pi/180}" />
@@ -105,4 +105,5 @@
     </visual>
     <visual>
+      <origin xyz="0 0 -0.012" rpy="0 0 0"/>
       <geometry>
         <mesh filename="package://franka_pole/meshes/visual/2D_upper.dae"/>

Commit message: 2D pole redesign

File: robots/franka_pole.xacro (robot description, xacro)
@@ -44,5 +44,5 @@
   <!-- Connection -->
   <joint name="$(arg arm_id)_pole_joint_connection" type="fixed">
-    <origin xyz="0.071 -0.071 0.03" rpy="${pi} 0 ${-pi/4}" />
+    <origin xyz="${0.085/sqrt(2)} -${0.085/sqrt(2)} 0.03" rpy="${pi} 0 ${-pi/4}" />
     <parent link="$(arg arm_id)_link8" />
     <child  link="$(arg arm_id)_pole_link_lower" />
@@ -70,5 +70,5 @@
     <origin xyz="0 0 0" rpy="0 0 0"/>
     <axis xyz="1 0 0"/>
-    <limit velocity="1000000" lower="${-20*pi/180}" effort="0" upper="${20*pi/180}" />
+    <limit velocity="1000000" lower="${-15*pi/180}" effort="0" upper="${15*pi/180}" />
     <dynamics damping="0.0"/>
   </joint>

File: robots/franka_pole_2D.xacro (robot description, xacro)
@@ -45,5 +45,5 @@
   <!-- Connection -->
   <joint name="$(arg arm_id)_pole_joint_connection" type="fixed">
-    <origin xyz="0.071 -0.071 0.0" rpy="${pi} 0 ${-pi/4}" />
+    <origin xyz="${0.110/sqrt(2)} -${0.110/sqrt(2)} 0.03" rpy="${pi} 0 ${-pi/4}" />
     <parent link="$(arg arm_id)_link8" />
     <child  link="$(arg arm_id)_pole_link_lower" />
@@ -71,5 +71,5 @@
     <origin xyz="0 0 0" rpy="0 0 0"/>
     <axis xyz="0 1 0"/>
-    <limit velocity="1000000" lower="${-20*pi/180}" effort="0" upper="${20*pi/180}" />
+    <limit velocity="1000000" lower="${15*pi/180}" effort="0" upper="${45*pi/180}" />
     <dynamics damping="0.0"/>
   </joint>
@@ -77,5 +77,5 @@
   <link name="$(arg arm_id)_pole_link_middle">
     <visual>
-      <origin xyz="0 0 0" rpy="0 0 0"/>
+      <origin xyz="0 0 0" rpy="0 ${-pi/6} 0"/>
       <geometry>
         <mesh filename="package://franka_pole/meshes/visual/2D_middle.dae"/>
@@ -96,5 +96,5 @@
     <origin xyz="0 0 0.012" rpy="0 0 0"/>
     <axis xyz="1 0 0"/>
-    <limit velocity="1000000" lower="${-20*pi/180}" effort="0" upper="${20*pi/180}" />
+    <limit velocity="1000000" lower="${-15*pi/180}" effort="0" upper="${15*pi/180}" />
     <dynamics damping="0.0"/>
   </joint>
@@ -108,5 +108,5 @@
     </visual>
     <visual>
-      <origin xyz="0 0 -0.012" rpy="0 0 0"/>
+      <origin xyz="0 0 -0.012" rpy="0 ${-pi/6} 0"/>
       <geometry>
         <mesh filename="package://franka_pole/meshes/visual/2D_upper.dae"/>

Commit message: Refactoring (plotter not working)

File: robots/franka_pole.xacro (robot description, xacro)
@@ -36,9 +36,9 @@
   <!-- Pendulum -->
   <xacro:property name="lower_mass" value="0.5" />
-  <xacro:property name="upper_mass" value="0.1" />
+  <xacro:property name="upper_mass" value="0.05" />
   <xacro:property name="ball_mass" value="0.1" />
-  <xacro:property name="beam_mass" value="0.05" />
-  <xacro:property name="beam_length" value="0.6" />
-  <xacro:property name="beam_radius" value="0.01" />
+  <xacro:property name="beam_mass" value="0.01" />
+  <xacro:property name="beam_length" value="0.5" />
+  <xacro:property name="beam_radius" value="0.005" />
   <xacro:property name="ball_radius" value="0.05" />
   <!-- Connection -->
@@ -70,5 +70,5 @@
     <origin xyz="0 0 0" rpy="0 0 0"/>
     <axis xyz="1 0 0"/>
-    <limit velocity="1000000" lower="${-15*pi/180}" effort="0" upper="${15*pi/180}" />
+    <limit velocity="1000000" lower="${-10*pi/180}" effort="0" upper="${10*pi/180}" />
     <dynamics damping="0.0"/>
   </joint>
@@ -88,5 +88,5 @@
     <inertial>
       <origin xyz="0 0 ${beam_length/2.0}" rpy="0 0 0"/>
-      <mass value="${beam_mass}"/>
+      <mass value="${upper_mass} + ${beam_mass}"/>
       <inertia
       ixx="${beam_mass * beam_length*beam_length / 12.0 + beam_mass * beam_radius*beam_radius / 4.0}" ixy="0.0" ixz="0.0"

File: robots/franka_pole_2D.xacro (robot description, xacro)
@@ -39,7 +39,7 @@
   <xacro:property name="upper_mass" value="0.1" />
   <xacro:property name="ball_mass" value="0.1" />
-  <xacro:property name="beam_mass" value="0.05" />
-  <xacro:property name="beam_length" value="0.6" />
-  <xacro:property name="beam_radius" value="0.01" />
+  <xacro:property name="beam_mass" value="0.01" />
+  <xacro:property name="beam_length" value="0.5" />
+  <xacro:property name="beam_radius" value="0.005" />
   <xacro:property name="ball_radius" value="0.05" />
   <!-- Connection -->
@@ -71,5 +71,5 @@
     <origin xyz="0 0 0" rpy="0 0 0"/>
     <axis xyz="0 1 0"/>
-    <limit velocity="1000000" lower="${15*pi/180}" effort="0" upper="${45*pi/180}" />
+    <limit velocity="1000000" lower="${-10*pi/180}" effort="0" upper="${10*pi/180}" />
     <dynamics damping="0.0"/>
   </joint>
@@ -96,5 +96,5 @@
     <origin xyz="0 0 0.012" rpy="0 0 0"/>
     <axis xyz="1 0 0"/>
-    <limit velocity="1000000" lower="${-15*pi/180}" effort="0" upper="${15*pi/180}" />
+    <limit velocity="1000000" lower="${-10*pi/180}" effort="0" upper="${10*pi/180}" />
     <dynamics damping="0.0"/>
   </joint>
@@ -115,5 +115,5 @@
     <inertial>
       <origin xyz="0 0 ${beam_length/2.0}" rpy="0 0 0"/>
-      <mass value="${beam_mass}"/>
+      <mass value="${upper_mass} + ${beam_mass}"/>
       <inertia
       ixx="${beam_mass * beam_length*beam_length / 12.0 + beam_mass * beam_radius*beam_radius / 4.0}" ixy="0.0" ixz="0.0"

Commit message: Bugfixes

File: robots/franka_pole.xacro (robot description, xacro)
@@ -41,5 +41,5 @@
   <xacro:property name="beam_length" value="0.5" />
   <xacro:property name="beam_radius" value="0.005" />
-  <xacro:property name="ball_radius" value="0.05" />
+  <xacro:property name="ball_radius" value="0.025" />
   <!-- Connection -->
   <joint name="$(arg arm_id)_pole_joint_connection" type="fixed">
@@ -70,5 +70,5 @@
     <origin xyz="0 0 0" rpy="0 0 0"/>
     <axis xyz="1 0 0"/>
-    <limit velocity="1000000" lower="${-10*pi/180}" effort="0" upper="${10*pi/180}" />
+    <limit velocity="1000000" lower="${-30*pi/180}" effort="0" upper="${30*pi/180}" />
     <dynamics damping="0.0"/>
   </joint>

File: robots/franka_pole_2D.xacro (robot description, xacro)
@@ -42,5 +42,5 @@
   <xacro:property name="beam_length" value="0.5" />
   <xacro:property name="beam_radius" value="0.005" />
-  <xacro:property name="ball_radius" value="0.05" />
+  <xacro:property name="ball_radius" value="0.025" />
   <!-- Connection -->
   <joint name="$(arg arm_id)_pole_joint_connection" type="fixed">

Commit message: LQR implemented, model improved

File: robots/franka_pole.xacro (robot description, xacro)
@@ -34,12 +34,4 @@
     <self_collide>true</self_collide>
   </gazebo>
-  <!-- Pendulum -->
-  <xacro:property name="lower_mass" value="0.5" />
-  <xacro:property name="upper_mass" value="0.05" />
-  <xacro:property name="ball_mass" value="0.1" />
-  <xacro:property name="beam_mass" value="0.01" />
-  <xacro:property name="beam_length" value="0.5" />
-  <xacro:property name="beam_radius" value="0.005" />
-  <xacro:property name="ball_radius" value="0.025" />
   <!-- Connection -->
   <joint name="$(arg arm_id)_pole_joint_connection" type="fixed">
@@ -48,5 +40,5 @@
     <child  link="$(arg arm_id)_pole_link_lower" />
   </joint>
-  <!-- Lower bearing -->
+  <!-- Lower bearing and holder -->
   <link name="$(arg arm_id)_pole_link_lower">
     <visual>
@@ -57,10 +49,10 @@
     </visual>
     <inertial>
-      <origin xyz="0 0 0" rpy="0 0 0"/>
-      <mass value="${lower_mass}"/>
+      <origin xyz="-0.029999510887629054 0.0 -0.0756128079743589" rpy="0 0 0"/>
+      <mass value="1.3331586494006493"/>
       <inertia
-      ixx="0.0" ixy="0.0" ixz="0.0"
-      iyy="0.0" iyz="0.0"
-      izz="0.0"/>
+      ixx="0.0014326187365418066" ixy="0.0" ixz="-0.00018436642795335555"
+      iyy="0.002670317415952603" iyz="0.0"
+      izz="0.0022496803634875807"/>
     </inertial>
   </link>
@@ -73,46 +65,31 @@
     <dynamics damping="0.0"/>
   </joint>
-  <!-- Upper bearing and beam -->
+  <!-- Upper bearing, beam  and ball -->
   <link name="$(arg arm_id)_pole_link_upper">
     <visual>
-      <origin xyz="0 0 ${beam_length/2.0 + 0.03}" rpy="0 0 0"/>
-      <geometry>
-        <cylinder length="${beam_length - 0.06}" radius = "${beam_radius}"/>
-      </geometry>
-    </visual>
-    <visual>
+      <origin xyz="0 0 0" rpy="0 0 0"/>
       <geometry>
         <mesh filename="package://franka_pole/meshes/visual/1D_upper.dae"/>
       </geometry>
     </visual>
-    <inertial>
-      <origin xyz="0 0 ${beam_length/2.0}" rpy="0 0 0"/>
-      <mass value="${upper_mass} + ${beam_mass}"/>
-      <inertia
-      ixx="${beam_mass * beam_length*beam_length / 12.0 + beam_mass * beam_radius*beam_radius / 4.0}" ixy="0.0" ixz="0.0"
-      iyy="${beam_mass * beam_length*beam_length / 12.0 + beam_mass * beam_radius*beam_radius / 4.0}" iyz="0.0"
-      izz="${beam_mass * beam_radius*beam_radius / 2.0}"/>
-    </inertial>
-  </link>
-  <joint name="$(arg arm_id)_pole_joint_ball" type="fixed">
-    <parent link="$(arg arm_id)_pole_link_upper"/>
-    <child link="$(arg arm_id)_pole_link_ball"/>
-    <origin xyz="0 0 ${beam_length}" rpy="0 0 0"/>
-  </joint>
-  <!-- Ball -->
-  <link name="$(arg arm_id)_pole_link_ball">
     <visual>
-      <origin xyz="0 0 0" rpy="0 0 0"/>
+      <origin xyz="0 0 ${0.65/2 + 0.06}" rpy="0 0 0"/>
       <geometry>
-        <sphere radius = "${ball_radius}"/>
+        <cylinder length="0.65" radius="0.005"/>
+      </geometry>
+    </visual>
+    <visual>
+      <origin xyz="0 0 0.43" rpy="0 0 0"/>
+      <geometry>
+        <sphere radius="0.0275"/>
       </geometry>
     </visual>
     <inertial>
-      <origin xyz="0 0 0" rpy="0 0 0"/>
-      <mass value="${ball_mass}"/>
+      <origin xyz="0.0 0.0 0.1645383811058607" rpy="0 0 0"/>
+      <mass value="0.31834554992177827"/>
       <inertia
-      ixx="${2.0 * ball_mass * ball_radius*ball_radius / 5.0}" ixy="0.0" ixz="0.0"
-      iyy="${2.0 * ball_mass * ball_radius*ball_radius / 5.0}" iyz="0.0"
-      izz="${2.0 * ball_mass * ball_radius*ball_radius / 5.0}"/>
+      ixx="0.01035842720256339" ixy="0.0" ixz="0.0"
+      iyy="0.010233978160578083" iyz="0.0"
+      izz="0.0002389493708066703"/>
     </inertial>
   </link>

File: robots/franka_pole_2D.xacro (robot description, xacro)
@@ -34,13 +34,4 @@
     <self_collide>true</self_collide>
   </gazebo>
-  <!-- Pendulum -->
-  <xacro:property name="lower_mass" value="0.5" />
-  <xacro:property name="middle_mass" value="0.05" />
-  <xacro:property name="upper_mass" value="0.1" />
-  <xacro:property name="ball_mass" value="0.1" />
-  <xacro:property name="beam_mass" value="0.01" />
-  <xacro:property name="beam_length" value="0.5" />
-  <xacro:property name="beam_radius" value="0.005" />
-  <xacro:property name="ball_radius" value="0.025" />
   <!-- Connection -->
   <joint name="$(arg arm_id)_pole_joint_connection" type="fixed">
@@ -58,10 +49,10 @@
     </visual>
     <inertial>
-      <origin xyz="0 0 0" rpy="0 0 0"/>
-      <mass value="${lower_mass}"/>
+      <origin xyz="-0.05109889873590216 2.087955225371467e-05 -0.09641756504956266" rpy="0 0 0"/>
+      <mass value="0.3291666816221097"/>
       <inertia
-      ixx="0.0" ixy="0.0" ixz="0.0"
-      iyy="0.0" iyz="0.0"
-      izz="0.0"/>
+      ixx="0.0019391504246096141" ixy="-1.2810025473031176e-07" ixz="-0.00018658257593334764"
+      iyy="0.0032282596099721715" iyz="-2.76251743233805e-07"
+      izz="0.002428110536000401"/>
     </inertial>
   </link>
@@ -77,5 +68,5 @@
   <link name="$(arg arm_id)_pole_link_middle">
     <visual>
-      <origin xyz="0 0 0" rpy="0 ${-pi/6} 0"/>
+      <origin xyz="0 0 0" rpy="0 0 0"/>
       <geometry>
         <mesh filename="package://franka_pole/meshes/visual/2D_middle.dae"/>
@@ -83,10 +74,10 @@
     </visual>
     <inertial>
-      <origin xyz="0 0 0" rpy="0 0 0"/>
-      <mass value="${middle_mass}"/>
+      <origin xyz="0.0 6.359054534633294e-09 0.006000000469716085" rpy="0 0 0"/>
+      <mass value="0.01583948395827795"/>
       <inertia
-      ixx="0.0" ixy="0.0" ixz="0.0"
-      iyy="0.0" iyz="0.0"
-      izz="0.0"/>
+      ixx="2.2608411674142452e-05" ixy="0.0" ixz="0.0"
+      iyy="2.2608411674142462e-05" iyz="0.0"
+      izz="1.612722485663805e-05"/>
     </inertial>
   </link>
@@ -99,47 +90,31 @@
     <dynamics damping="0.0"/>
   </joint>
-  <!-- Upper bearing and beam -->
+  <!-- Upper bearing, beam and ball -->
   <link name="$(arg arm_id)_pole_link_upper">
     <visual>
-      <origin xyz="0 0 ${beam_length/2.0 + 0.03}" rpy="0 0 0"/>
-      <geometry>
-        <cylinder length="${beam_length - 0.06}" radius = "${beam_radius}"/>
-      </geometry>
-    </visual>
-    <visual>
-      <origin xyz="0 0 -0.012" rpy="0 ${-pi/6} 0"/>
+      <origin xyz="0 0 -0.012" rpy="0 0 0"/>
       <geometry>
         <mesh filename="package://franka_pole/meshes/visual/2D_upper.dae"/>
       </geometry>
     </visual>
-    <inertial>
-      <origin xyz="0 0 ${beam_length/2.0}" rpy="0 0 0"/>
-      <mass value="${upper_mass} + ${beam_mass}"/>
-      <inertia
-      ixx="${beam_mass * beam_length*beam_length / 12.0 + beam_mass * beam_radius*beam_radius / 4.0}" ixy="0.0" ixz="0.0"
-      iyy="${beam_mass * beam_length*beam_length / 12.0 + beam_mass * beam_radius*beam_radius / 4.0}" iyz="0.0"
-      izz="${beam_mass * beam_radius*beam_radius / 2.0}"/>
-    </inertial>
-  </link>
-  <joint name="$(arg arm_id)_pole_joint_ball" type="fixed">
-    <parent link="$(arg arm_id)_pole_link_upper"/>
-    <child link="$(arg arm_id)_pole_link_ball"/>
-    <origin xyz="0 0 ${beam_length}" rpy="0 0 0"/>
-  </joint>
-  <!-- Ball -->
-  <link name="$(arg arm_id)_pole_link_ball">
     <visual>
-      <origin xyz="0 0 0" rpy="0 0 0"/>
+      <origin xyz="0 0 ${0.06 + 0.65/2}" rpy="0 0 0"/>
       <geometry>
-        <sphere radius = "${ball_radius}"/>
+        <cylinder length="0.65" radius = "0.005"/>
+      </geometry>
+    </visual>
+    <visual>
+      <origin xyz="0 0 0.43" rpy="0 0 0"/>
+      <geometry>
+        <sphere radius = "0.00275"/>
       </geometry>
     </visual>
     <inertial>
-      <origin xyz="0 0 0" rpy="0 0 0"/>
-      <mass value="${ball_mass}"/>
+      <origin xyz="-7.652676027542849e-05 3.225024691385294e-07 ${0.13021144099656237 - 0.012}" rpy="0 0 0"/>
+      <mass value="0.11035793369531807"/>
       <inertia
-      ixx="${2.0 * ball_mass * ball_radius*ball_radius / 5.0}" ixy="0.0" ixz="0.0"
-      iyy="${2.0 * ball_mass * ball_radius*ball_radius / 5.0}" iyz="0.0"
-      izz="${2.0 * ball_mass * ball_radius*ball_radius / 5.0}"/>
+      ixx="0.00312322181055378" ixy="0.0" ixz="-5.323303220087574e-07"
+      iyy="0.002922973095088403" iyz="4.395839128943858e-09"
+      izz="0.00036214355788495307"/>
     </inertial>
   </link>

Commit message: Minor changes

File: robots/franka_pole.xacro (robot description, xacro)
@@ -86,10 +86,10 @@
     </visual>
     <inertial>
-      <origin xyz="0.0 0.0 0.1645383811058607" rpy="0 0 0"/>
-      <mass value="0.31834554992177827"/>
+      <origin xyz="0.0 0.0 0.18292189266626382" rpy="0 0 0"/>
+      <mass value="0.34291554992177825"/>
       <inertia
-      ixx="0.01035842720256339" ixy="0.0" ixz="0.0"
-      iyy="0.010233978160578083" iyz="0.0"
-      izz="0.0002389493708066703"/>
+      ixx="0.012404643041130634" ixy="0.0" ixz="0.0"
+      iyy="0.012280193999145327" iyz="0.0"
+      izz="0.00023956362080667035"/>
     </inertial>
   </link>

File: robots/franka_pole_2Db.xacro (robot description, xacro)
@@ -49,10 +49,10 @@
     </visual>
     <inertial>
-      <origin xyz="0.0 -0.03161502390972815 -0.06659192458617054" rpy="0 0 0"/>
-      <mass value="0.27322280135974475"/>
+      <origin xyz="-0.031615023280958485 0.0 -0.06659192458617054" rpy="0 0 0"/>
+      <mass value="0.2732228013597448"/>
       <inertia
-      ixx="0.0028058366276666187" ixy="0.0" ixz="0.0"
-      iyy="0.0016993982151537815" iyz="-8.877913787029444e-05"
-      izz="0.002116794356382879"/>
+      ixx="0.0016993982151537815" ixy="0.0" ixz="-8.877913625404171e-05"
+      iyy="0.00280583662568493" iyz="0.0"
+      izz="0.002116794354401193"/>
     </inertial>
   </link>
@@ -68,6 +68,10 @@
   <link name="$(arg arm_id)_pole_link_middle">
     <inertial>
-      <origin xyz="0.0 0.0 0.0" rpy="0 0 0"/>
+      <origin xyz="0 0 0.005" rpy="0 0 0"/>
       <mass value="0.001"/>
+      <inertia
+      ixx="1e-05" ixy="0.0" ixz="0.0"
+      iyy="1e-05" iyz="0.0"
+      izz="1e-05"/>
     </inertial>
   </link>
@@ -75,5 +79,5 @@
     <parent link="$(arg arm_id)_pole_link_middle"/>
     <child link="$(arg arm_id)_pole_link_upper"/>
-    <origin xyz="0 0 0" rpy="0 0 0"/>
+    <origin xyz="0 0 0.01" rpy="0 0 0"/>
     <axis xyz="1 0 0"/>
     <limit velocity="1000000" lower="${-30*pi/180}" effort="0" upper="${30*pi/180}" />
@@ -83,5 +87,5 @@
   <link name="$(arg arm_id)_pole_link_upper">
     <visual>
-      <origin xyz="0 0 0" rpy="0 0 0"/>
+      <origin xyz="0 0 -0.01" rpy="0 0 0"/>
       <geometry>
         <mesh filename="package://franka_pole/meshes/visual/2Db_upper.dae"/>
@@ -89,16 +93,16 @@
     </visual>
     <visual>
-      <origin xyz="0 0 ${0.039 + 0.5/2}" rpy="0 0 0"/>
+      <origin xyz="0 0 ${0.039 + 0.65/2 - 0.01}" rpy="0 0 0"/>
       <geometry>
-        <cylinder length="0.5" radius="0.005"/>
+        <cylinder length="0.65" radius="0.005"/>
       </geometry>
     </visual>
     <inertial>
-      <origin xyz="0.0 0.0 0.35075520003248506" rpy="0 0 0"/>
-      <mass value="0.03241958003770816"/>
+      <origin xyz="0.0 0.0 ${0.43117306006864087 - 0.01}" rpy="0 0 0"/>
+      <mass value="0.038719580037708166"/>
       <inertia
-      ixx="0.001036931649741803" ixy="0.0" ixz="0.0"
-      iyy="0.001036931649741803" iyz="0.0"
-      izz="1.109395012820758e-05"/>
+      ixx="0.0019970733076910907" ixy="0.0" ixz="0.0"
+      iyy="0.0019970733076910907" iyz="0.0"
+      izz="1.1251450128207583e-05"/>
     </inertial>
   </link>
