Commit message: Small fixes, adaptation to reality

File: robots/franka_pole.xacro (robot description, xacro)
@@ -49,10 +49,10 @@
     </visual>
     <inertial>
-      <origin xyz="-0.029999510887629054 0.0 -0.0756128079743589" rpy="0 0 0"/>
-      <mass value="1.3331586494006493"/>
+      <origin xyz="-0.022003229638627025 0.0 -0.06809318358207639" rpy="0 0 0"/>
+      <mass value="0.5054569600898893"/>
       <inertia
-      ixx="0.0014326187365418066" ixy="0.0" ixz="-0.00018436642795335555"
-      iyy="0.002670317415952603" iyz="0.0"
-      izz="0.0022496803634875807"/>
+      ixx="0.0008334988699267267" ixy="0.0" ixz="-0.00013466959040378683"
+      iyy="0.0013231310073701067" iyz="0.0"
+      izz="0.0008994724071810742"/>
     </inertial>
   </link>
@@ -89,7 +89,7 @@
       <mass value="0.34291554992177825"/>
       <inertia
-      ixx="0.012404643041130634" ixy="0.0" ixz="0.0"
-      iyy="0.012280193999145327" iyz="0.0"
-      izz="0.00023956362080667035"/>
+      ixx="0.012455943363405825" ixy="0.0" ixz="0.0"
+      iyy="0.012294411551671247" iyz="0.0"
+      izz="0.00027958843954040385"/>
     </inertial>
   </link>

File: robots/franka_pole_2D.xacro (robot description, xacro)
@@ -49,10 +49,10 @@
     </visual>
     <inertial>
-      <origin xyz="-0.05109889873590216 2.087955225371467e-05 -0.09641756504956266" rpy="0 0 0"/>
-      <mass value="0.3291666816221097"/>
+      <origin xyz="-0.05417692376165083 1.631629415101512e-05 -0.10102516335402327" rpy="0 0 0"/>
+      <mass value="0.42122634375995777"/>
       <inertia
-      ixx="0.0019391504246096141" ixy="-1.2810025473031176e-07" ixz="-0.00018658257593334764"
-      iyy="0.0032282596099721715" iyz="-2.76251743233805e-07"
-      izz="0.002428110536000401"/>
+      ixx="0.0009355660559119161" ixy="-1.919376506548452e-07" ixz="-0.00024073219427997694"
+      iyy="0.0014466958209361893" iyz="-3.8184740643923794e-07"
+      izz="0.0009820861200053165"/>
     </inertial>
   </link>
@@ -77,7 +77,7 @@
       <mass value="0.01583948395827795"/>
       <inertia
-      ixx="2.2608411674142452e-05" ixy="0.0" ixz="0.0"
-      iyy="2.2608411674142462e-05" iyz="0.0"
-      izz="1.612722485663805e-05"/>
+      ixx="5.652102918535614e-06" ixy="0.0" ixz="0.0"
+      iyy="5.652102918535616e-06" iyz="0.0"
+      izz="4.031806214159512e-06"/>
     </inertial>
   </link>
@@ -114,7 +114,7 @@
       <mass value="0.13492793369531808"/>
       <inertia
-      ixx="0.005511654978105017" ixy="0.0" ixz="-9.981512278924966e-07"
-      iyy="0.005311406380325907" iyz="6.358922261996068e-09"
-      izz="0.00036275792557540116"/>
+      ixx="0.005252713974715477" ixy="0.0" ixz="-1.0207840204095797e-06"
+      iyy="0.005226062508314185" iyz="5.116218503426479e-09"
+      izz="0.00014648155653184902"/>
     </inertial>
   </link>

File: robots/franka_pole_2Db.xacro (robot description, xacro)
@@ -49,10 +49,10 @@
     </visual>
     <inertial>
-      <origin xyz="-0.031615023280958485 0.0 -0.06659192458617054" rpy="0 0 0"/>
-      <mass value="0.2732228013597448"/>
+      <origin xyz="-0.029498584051831502 0.0 -0.06313961580055441" rpy="0 0 0"/>
+      <mass value="0.41100000000000003"/>
       <inertia
-      ixx="0.0016993982151537815" ixy="0.0" ixz="-8.877913625404171e-05"
-      iyy="0.00280583662568493" iyz="0.0"
-      izz="0.002116794354401193"/>
+      ixx="0.000895475019378853" ixy="0.0" ixz="-0.00015591824406532102"
+      iyy="0.0013577361299841326" iyz="0.0"
+      izz="0.0008258336095097959"/>
     </inertial>
   </link>
@@ -84,5 +84,5 @@
     <dynamics damping="0.0"/>
   </joint>
-  <!-- Upper bearing, beam and ball -->
+  <!-- Upper bearing, beam, pine and ball -->
   <link name="$(arg arm_id)_pole_link_upper">
     <visual>
@@ -95,14 +95,20 @@
       <origin xyz="0 0 ${0.039 + 0.65/2 - 0.01}" rpy="0 0 0"/>
       <geometry>
+        <sphere radius="0.0275"/>
+      </geometry>
+    </visual>
+    <visual>
+      <origin xyz="0 0 ${0.039 + 0.65/2 - 0.01}" rpy="0 0 0"/>
+      <geometry>
         <cylinder length="0.65" radius="0.005"/>
       </geometry>
     </visual>
     <inertial>
-      <origin xyz="0.0 0.0 ${0.43117306006864087 - 0.01}" rpy="0 0 0"/>
-      <mass value="0.038719580037708166"/>
+      <origin xyz="0.0 0.0 ${0.4632543529459209 - 0.01}" rpy="0 0 0"/>
+      <mass value="0.1593"/>
       <inertia
-      ixx="0.0019970733076910907" ixy="0.0" ixz="0.0"
-      iyy="0.0019970733076910907" iyz="0.0"
-      izz="1.1251450128207583e-05"/>
+      ixx="0.012139364109265307" ixy="0.0" ixz="0.0"
+      iyy="0.012139364109265307" iyz="0.0"
+      izz="4.63115872630246e-05"/>
     </inertial>
   </link>

Commit message: Refactoring, parameters improved (unstable)

File: robots/franka_pole.xacro (robot description, xacro)
@@ -34,72 +34,3 @@
     <self_collide>true</self_collide>
   </gazebo>
-  <!-- Connection -->
-  <joint name="$(arg arm_id)_pole_joint_connection" type="fixed">
-    <origin xyz="${0.085/sqrt(2)} -${0.085/sqrt(2)} 0.03" rpy="${pi} 0 ${-pi/4}" />
-    <parent link="$(arg arm_id)_link8" />
-    <child  link="$(arg arm_id)_pole_link_lower" />
-  </joint>
-  <!-- Lower bearing and holder -->
-  <link name="$(arg arm_id)_pole_link_lower">
-    <visual>
-      <origin xyz="0 0 0" rpy="0 0 0"/>
-      <geometry>
-        <mesh filename="package://franka_pole/meshes/visual/1D_lower.dae"/>
-      </geometry>
-    </visual>
-    <inertial>
-      <origin xyz="-0.022003229638627025 0.0 -0.06809318358207639" rpy="0 0 0"/>
-      <mass value="0.5054569600898893"/>
-      <inertia
-      ixx="0.0008334988699267267" ixy="0.0" ixz="-0.00013466959040378683"
-      iyy="0.0013231310073701067" iyz="0.0"
-      izz="0.0008994724071810742"/>
-    </inertial>
-  </link>
-  <joint name="$(arg arm_id)_pole_joint_x" type="revolute">
-    <parent link="$(arg arm_id)_pole_link_lower"/>
-    <child link="$(arg arm_id)_pole_link_upper"/>
-    <origin xyz="0 0 0" rpy="0 0 0"/>
-    <axis xyz="1 0 0"/>
-    <limit velocity="1000000" lower="${-30*pi/180}" effort="0" upper="${30*pi/180}" />
-    <dynamics damping="0.0"/>
-  </joint>
-  <!-- Upper bearing, beam  and ball -->
-  <link name="$(arg arm_id)_pole_link_upper">
-    <visual>
-      <origin xyz="0 0 0" rpy="0 0 0"/>
-      <geometry>
-        <mesh filename="package://franka_pole/meshes/visual/1D_upper.dae"/>
-      </geometry>
-    </visual>
-    <visual>
-      <origin xyz="0 0 ${0.65/2 + 0.06}" rpy="0 0 0"/>
-      <geometry>
-        <cylinder length="0.65" radius="0.005"/>
-      </geometry>
-    </visual>
-    <visual>
-      <origin xyz="0 0 0.43" rpy="0 0 0"/>
-      <geometry>
-        <sphere radius="0.0275"/>
-      </geometry>
-    </visual>
-    <inertial>
-      <origin xyz="0.0 0.0 0.18292189266626382" rpy="0 0 0"/>
-      <mass value="0.34291554992177825"/>
-      <inertia
-      ixx="0.012455943363405825" ixy="0.0" ixz="0.0"
-      iyy="0.012294411551671247" iyz="0.0"
-      izz="0.00027958843954040385"/>
-    </inertial>
-  </link>
-  <transmission name="$(arg arm_id)_pole_joint_x_transmission">
-    <type>transmission_interface/SimpleTransmission</type>
-    <joint name="$(arg arm_id)_pole_joint_x">
-      <hardwareInterface>hardware_interface/PositionJointInterface</hardwareInterface>
-    </joint>
-    <actuator name="$(arg arm_id)_pole_joint_x_motor">
-      <hardwareInterface>hardware_interface/PositionJointInterface</hardwareInterface>
-    </actuator>
-  </transmission>
 </robot>

Commit message: 2Dc model added, calibrator added, little refactoring

File: robots/franka_pole.xacro (robot description, xacro)
@@ -2,7 +2,13 @@
 <robot xmlns:xacro="http://www.ros.org/wiki/xacro" name="franka_pole">
   <xacro:arg name="arm_id" default="panda" />
+  <xacro:arg name="friction" default="false" />
   <!-- Create a simulatable URDF -->
   <xacro:include filename="$(find franka_description)/robots/utils.xacro" />
-  <xacro:include filename="$(find franka_pole)/robots/panda_gazebo.xacro" />
+  <xacro:unless value="$(arg friction)">
+    <xacro:include filename="$(find franka_pole)/robots/panda_gazebo.xacro" />
+  </xacro:unless>
+  <xacro:if value="$(arg friction)">
+    <xacro:include filename="$(find franka_description)/robots/panda_gazebo.xacro" />
+  </xacro:if>
   <xacro:panda_arm arm_id="$(arg arm_id)" />
   <xacro:hand arm_id="$(arg arm_id)" rpy="0 0 ${-pi/4}" connected_to="$(arg arm_id)_link8" />

File: robots/franka_pole_1D.xacro (robot description, xacro)
@@ -2,7 +2,13 @@
 <robot xmlns:xacro="http://www.ros.org/wiki/xacro" name="franka_pole">
   <xacro:arg name="arm_id" default="panda" />
+  <xacro:arg name="friction" default="false" />
   <!-- Create a simulatable URDF -->
   <xacro:include filename="$(find franka_description)/robots/utils.xacro" />
-  <xacro:include filename="$(find franka_pole)/robots/panda_gazebo.xacro" />
+  <xacro:unless value="$(arg friction)">
+    <xacro:include filename="$(find franka_pole)/robots/panda_gazebo.xacro" />
+  </xacro:unless>
+  <xacro:if value="$(arg friction)">
+    <xacro:include filename="$(find franka_description)/robots/panda_gazebo.xacro" />
+  </xacro:if>
   <xacro:panda_arm arm_id="$(arg arm_id)" />
   <xacro:hand arm_id="$(arg arm_id)" rpy="0 0 ${-pi/4}" connected_to="$(arg arm_id)_link8" />

File: robots/franka_pole_2D.xacro (robot description, xacro)
@@ -2,7 +2,13 @@
 <robot xmlns:xacro="http://www.ros.org/wiki/xacro" name="franka_pole">
   <xacro:arg name="arm_id" default="panda" />
+  <xacro:arg name="friction" default="false" />
   <!-- Create a simulatable URDF -->
   <xacro:include filename="$(find franka_description)/robots/utils.xacro" />
-  <xacro:include filename="$(find franka_pole)/robots/panda_gazebo.xacro" />
+  <xacro:unless value="$(arg friction)">
+    <xacro:include filename="$(find franka_pole)/robots/panda_gazebo.xacro" />
+  </xacro:unless>
+  <xacro:if value="$(arg friction)">
+    <xacro:include filename="$(find franka_description)/robots/panda_gazebo.xacro" />
+  </xacro:if>
   <xacro:panda_arm arm_id="$(arg arm_id)" />
   <xacro:hand arm_id="$(arg arm_id)" rpy="0 0 ${-pi/4}" connected_to="$(arg arm_id)_link8" />

File: robots/franka_pole_2Dc.xacro (robot description, xacro)
@@ -51,5 +51,5 @@
       <origin xyz="0 0 0" rpy="0 0 0"/>
       <geometry>
-        <mesh filename="package://franka_pole/meshes/visual/2Db_lower.dae"/>
+        <mesh filename="package://franka_pole/meshes/visual/2Dc_lower.dae"/>
       </geometry>
     </visual>
@@ -68,5 +68,5 @@
     <origin xyz="0 0 0" rpy="0 0 0"/>
     <axis xyz="0 1 0"/>
-    <limit velocity="1000000" lower="${-30*pi/180}" effort="0" upper="${30*pi/180}" />
+    <limit velocity="1000000" lower="${-60*pi/180}" effort="0" upper="${60*pi/180}" />
     <dynamics damping="0.0"/>
   </joint>
@@ -87,5 +87,5 @@
     <origin xyz="0 0 0.01" rpy="0 0 0"/>
     <axis xyz="1 0 0"/>
-    <limit velocity="1000000" lower="${-30*pi/180}" effort="0" upper="${30*pi/180}" />
+    <limit velocity="1000000" lower="${-60*pi/180}" effort="0" upper="${60*pi/180}" />
     <dynamics damping="0.0"/>
   </joint>
@@ -111,10 +111,10 @@
     </visual>
     <inertial>
-      <origin xyz="0.0 0.0 ${0.42771135304787394 - 0.01}" rpy="0 0 0"/>
+      <origin xyz="0.0 0.0 ${0.4632543529459209 - 0.01}" rpy="0 0 0"/>
       <mass value="0.1593"/>
       <inertia
-      ixx="0.013902072326225548" ixy="0.0" ixz="0.0"
-      iyy="0.013902072326225548" iyz="0.0"
-      izz="4.266992059635794e-05"/>
+      ixx="0.012139364109265307" ixy="0.0" ixz="0.0"
+      iyy="0.012139364109265307" iyz="0.0"
+      izz="4.63115872630246e-05"/>
     </inertial>
   </link>
